File: gameoflife.kicad_sch (KiCad schematic)
At the start: 8 parts, among them U1 74LS283, U2 74LS283, U3 74LS151, U4 74LS151, U5 74LS283, U6 74LS283, U7 74LS151, U8 74LS151

Commit message: changes
Parts:
- added U9: 74LS194, symbol 74xx:74LS194
Connections:
- net +5V: now also U9.16 (VCC)
- net GND: now also U9.8 (GND)
- net i11: now also U9.15 (Q0)
- net i12: now also U9.14 (Q1)
- net i21: now also U9.13 (Q2)
- net i22: now also U9.12 (Q3)
- removed net out: U3.5 (Z), U4.5 (Z), U7.5 (Z), U8.5 (Z)
- new net o11: U3.5 (Z), U9.3 (P0)
- new net o12: U7.5 (Z), U9.4 (P1)
- new net o21: U4.5 (Z), U9.5 (P2)
- new net o22: U8.5 (Z), U9.6 (P3)
